File: PCB/Fracture.kicad_sch (KiCad schematic)
At the start: 0 parts

Commit message: Schematic essentials
Parts:
- added BUZZER1: FST-1230, imported_components:BUZ-SMD_L12.0-W12.0_FUET-1230, symbol imported_components:FST-1230
- added C1: RVT1H470M0607, imported_components:CAP-SMD_BD6.3-L6.6-W6.6-LS7.6-FD, symbol imported_components:RVT1H470M0607
- added C10: 0.1uF, symbol Device:C
- added C19: RVT1E331M0810, imported_components:CAP-SMD_BD8.0-L8.3-W8.3-LS9.3-FD-1, symbol imported_components:RVT1E331M0810_C335985
- added C2, C3, C4, C5, C8, C9: 10uF, imported_components:C0805, symbol Device:C
- added C6, C7: 0.1uF, imported_components:C0805, symbol Device:C
- added D1, D2: SS54_C22452, imported_components:SMA_L4.4-W2.8-LS5.4-R-RD, symbol imported_components:SS54_C22452
- added D3: LED, imported_components:LED0805-RD, symbol Device:LED
- added H1, H2, H3, H4: MountingHole, MountingHole:MountingHole_3.2mm_M3_Pad_Via, symbol Mechanical:MountingHole
- added J1: Barrel_Jack, imported_components:DC-IN-TH_DC-005-A200, symbol Connector:Barrel_Jack_MountingPin
- added J2: Conn_01x02, imported_components:CONN-TH_P5.00_KF301-5.0-2P, symbol Connector:Conn_01x02_Pin
- added L1: CYA1040-33UH, imported_components:IND-SMD_L11.6-W10.1, symbol imported_components:CYA1040-33UH
- added L2: BLM21PG221SN1D, imported_components:L0805, symbol imported_components:BLM21PG221SN1D
- added P1: USB_C_Plug, imported_components:USB-C_SMD-TYPE-C-31-M-12, symbol Connector:USB_C_Plug
- added R1, R2: 10k, symbol Device:R
- added R3, R4: 5.1k, imported_components:R0805, symbol Device:R
- added R5, R6: 10k, imported_components:R0805, symbol Device:R
- added R7: 200, imported_components:R0805, symbol Device:R
- added R8, R9: 22, symbol Device:R
- added SW1, SW2: SW_Push, imported_components:SW-SMD_L3.9-W3.0-P4.45, symbol Switch:SW_Push
- added SW3: SW_SPDT, imported_components:SW-SMD_MST-12D18G4-SPDT-SLIDE-SWITCH, symbol Switch:SW_SPDT
- added U1: ESP32-S3-WROOM-1-N4, imported_components:WIFIM-SMD_ESP32-S3-WROOM-1-N8, symbol imported_components:ESP32-S3-WROOM-1-N4
- added U2: LM2596SX-5.0/NOPB, imported_components:TO-263-5_L10.2-W8.9-P1.70-TL, symbol imported_components:LM2596SX-5.0_NOPB
- added U3, U4: AMS1117-3.3, Package_TO_SOT_SMD:SOT-223-3_TabPin2, symbol Regulator_Linear:AMS1117-3.3
- added U5, U6: 74HC4067PW,118, imported_components:TSSOP-24_L7.8-W4.4-P0.65-LS6.4-BL, symbol imported_components:74HC4067PW,118
Connections:
- new net: D2.2 (K), L2.2
- new net: D3.2 (A), R7.2
- new net: D1.2 (K), L1.1, U2.2 (OUTPUT)
- new net: R1.1, U1.3 (EN)
- new net: R9.1, U1.14 (IO20)
- new net: P1.B5 (VCONN), R3.2
- new net: R8.2, U1.13 (IO19)
- new net: P1.A5 (CC), R4.1
- new net +3.3V: C10.1, C5.1, C7.1, R1.2, R2.2, R5.1, R6.1, R6.2, R7.1, SW2.1, U1.2 (3V3), U3.2 (VO)
- new net +3.3VA: C9.1, U4.2 (VO), U5.24 (VCC), U6.24 (VCC)
- new net +5V: C19.1, C3.1, C4.1, D2.1 (A), L1.2, U2.4 (FB), U3.3 (VI)
- new net +5VA: C8.1, L2.1, U4.3 (VI)
- new net +BATT: J1.1, J2.1 (Pin_1), SW3.3 (C)
- new net AM0: U5.1 (Z)
- new net AM0:0: U5.9 (Y0)
- new net AM0:1: U5.8 (Y1), U6.8 (Y1)
- new net AM0:10: U5.20 (Y11), U6.20 (Y11)
- new net AM0:11: U5.19 (Y12), U6.19 (Y12)
- new net AM0:12: U5.18 (Y13), U6.18 (Y13)
- new net AM0:13: U5.17 (Y14), U6.17 (Y14)
- new net AM0:14: U5.16 (Y15), U6.16 (Y15)
- new net AM0:2: U5.7 (Y2), U6.7 (Y2)
- new net AM0:3: U5.6 (Y3), U6.6 (Y3)
- new net AM0:4: U5.5 (Y4), U6.5 (Y4)
- new net AM0:5: U5.4 (Y5), U6.4 (Y5)
- new net AM0:6: U5.3 (Y6), U6.3 (Y6)
- new net AM0:7: U5.2 (Y7), U5.23 (Y8), U6.2 (Y7), U6.23 (Y8)
- new net AM0:8: U5.22 (Y9), U6.22 (Y9)
- new net AM0:9: U5.21 (Y10), U6.21 (Y10)
- new net AM1: U6.1 (Z)
- new net AM1:0: U6.9 (Y0)
- new net BUZZER_DATA: BUZZER1.1 (+)
- new net D+: P1.A6 (D+), R9.2
- new net D-: P1.A7 (D-), R8.1
- new net GND: BUZZER1.2, C1.2, C10.2, C19.2, C2.1, C3.2, C4.2, C5.2, C6.2, C7.2, C8.2, C9.2, D1.1 (A), D3.1 (K), J1.2, J1.MP (MountPin), J2.2 (Pin_2), P1.A1 (GND), P1.A12 (GND), P1.B1 (GND), P1.B12 (GND), P1.S1 (SHIELD), R3.1, R4.2, SW1.2, SW2.2, U1.1 (GND), U1.40 (GND), U1.41 (GND), U2.3 (GND), U2.5 (~{ON}/OFF), U2.6 (GND), U3.1 (GND), U4.1 (GND), U5.12 (GND), U5.15 (~{E}), U6.12 (GND), U6.15 (~{E})
- new net GPIO 0: C6.1, R2.1, R5.2, SW1.1, U1.27 (IO0)
- new net REG_BATT+: C1.1, C2.2, SW3.2 (B), U2.1 (VIN)
- new net SELECT0: U5.10 (S0), U6.10 (S0)
- new net SELECT1: U5.11 (S1), U6.11 (S1)
- new net SELECT2: U5.14 (S2), U6.14 (S2)
- new net SELECT3: U5.13 (S3), U6.13 (S3)
- new net VCC_5V: P1.A4 (VBUS), P1.A9 (VBUS), P1.B4 (VBUS), P1.B9 (VBUS)
- no-connect marks 0 -> 14
Other:
- note added: "Analog"
- note added: "BOOT"
- note added: "BUTTONS"
- note added: "MOUNTING"
- note added: "POWER"
- note added: "POWER LED"
- note added: "RST"
- note added: "SOUND"
- note added: "USB-C"
