File: PCB/Fracture.kicad_pcb (KiCad board)
At the start: 2 copper layers, 0 parts

Commit message: Schematic Done + PCB Layout Done
Parts:
- added BUZZER1: FST-1230, imported_components:BUZ-SMD_L12.0-W12.0_FUET-1230, B.Cu at (148.8, 72.8)
- added C1: 10uF, imported_components:C0805, B.Cu at (105.4, 46.0)
- added C10: 10uF, imported_components:C0805, B.Cu at (60.5, 54.7)
- added C11: 0.1uF, imported_components:C0805, B.Cu at (239.4, 28.2)
- added C12: 10uF, imported_components:C0805, B.Cu at (41.0, 48.6)
- added C13: RVT1E331M0810, imported_components:CAP-SMD_BD8.0-L8.3-W8.3-LS9.3-FD-1, B.Cu at (33.0, 55.0)
- added C14: 0.1uF, imported_components:C0805, B.Cu at (217.0, 58.4)
- added C15: 10uF, imported_components:C0805, B.Cu at (38.4, 40.8)
- added C16: 0.1uF, imported_components:C0805, B.Cu at (72.6, 40.8)
- added C17: 0.1uF, imported_components:C0805, B.Cu at (91.4, 40.8)
- added C18: 0.1uF, imported_components:C0805, B.Cu at (110.6, 40.6)
- added C19: 0.1uF, imported_components:C0805, B.Cu at (129.6, 40.8)
- added C2: 10uF, imported_components:C0805, B.Cu at (96.2, 51.4)
- added C20: 0.1uF, imported_components:C0805, B.Cu at (148.6, 40.8)
- added C21: 0.1uF, imported_components:C0805, B.Cu at (167.8, 40.8)
- added C22: 0.1uF, imported_components:C0805, B.Cu at (186.6, 40.8)
- added C23: 0.1uF, imported_components:C0805, B.Cu at (205.8, 40.8)
- added C24: 0.1uF, imported_components:C0805, B.Cu at (34.2, 69.4)
- added C25: 0.1uF, imported_components:C0805, B.Cu at (53.4, 69.4)
- added C26: 0.1uF, imported_components:C0805, B.Cu at (91.2, 69.4)
- added C27: 0.1uF, imported_components:C0805, B.Cu at (110.4, 69.4)
- added C28: 0.1uF, imported_components:C0805, B.Cu at (129.6, 69.4)
- added C29: 0.1uF, imported_components:C0805, B.Cu at (168.6, 69.4)
- added C3: 0.01uF, imported_components:C0805, B.Cu at (180.0, 45.2)
- added C30: 0.1uF, imported_components:C0805, B.Cu at (187.6, 69.4)
- added C31: 0.1uF, imported_components:C0805, B.Cu at (225.6, 69.4)
- added C32: 0.1uF, imported_components:C0805, B.Cu at (244.6, 69.4)
- added C33: 0.1uF, imported_components:C0805, B.Cu at (263.4, 69.4)
- added C34: 0.1uF, imported_components:C0805, B.Cu at (25.0, 88.4)
- added C35: 0.1uF, imported_components:C0805, B.Cu at (44.2, 88.4)
- added C36: 0.1uF, imported_components:C0805, B.Cu at (63.0, 88.4)
- added C37: 0.1uF, imported_components:C0805, B.Cu at (82.0, 88.4)
- added C38: 0.1uF, imported_components:C0805, B.Cu at (101.0, 88.4)
- added C39: 0.1uF, imported_components:C0805, B.Cu at (120.0, 88.4)
- added C4: 0.01uF, imported_components:C0805, B.Cu at (124.6, 45.6)
- added C40: 0.1uF, imported_components:C0805, B.Cu at (139.6, 88.4)
- added C41: 0.1uF, imported_components:C0805, B.Cu at (158.0, 88.4)
- added C42: 0.1uF, imported_components:C0805, B.Cu at (177.2, 88.4)
- added C43: 0.1uF, imported_components:C0805, B.Cu at (196.2, 88.4)
- added C44: 0.1uF, imported_components:C0805, B.Cu at (215.2, 88.4)
- added C45: 0.1uF, imported_components:C0805, B.Cu at (234.4, 88.4)
- added C46: 0.1uF, imported_components:C0805, B.Cu at (253.4, 88.4)
- added C47: 0.1uF, imported_components:C0805, B.Cu at (272.4, 88.4)
- added C48: 0.1uF, imported_components:C0805, B.Cu at (84.2, 48.0)
- added C49: 0.1uF, imported_components:C0805, B.Cu at (86.2, 49.4)
- added C5: 0.1uF, imported_components:C0805, B.Cu at (120.6, 47.6)
- added C50: 10uF, imported_components:C0805, B.Cu at (84.2, 52.0)
- added C51: 10uF, imported_components:C0805, B.Cu at (86.2, 53.6)
- added C52: 0.1uF, imported_components:C0805, B.Cu at (68.2, 40.2)
- added C53: 0.47uF, imported_components:C0805, B.Cu at (77.8, 53.4)
- added C54: 0.47uF, imported_components:C0805, B.Cu at (79.8, 53.4)
- added C55: 0.1uF, imported_components:C0805, B.Cu at (61.2, 46.4)
- added C56: 1uF, imported_components:C0805, B.Cu at (63.4, 46.4)
- added C57: 10uF, imported_components:C0805, B.Cu at (78.4, 67.6)
- added C58: 10uF, imported_components:C0805, B.Cu at (68.6, 69.6)
- added C59: RVT1V101M0607, imported_components:CAP-SMD_BD6.3-L6.6-W6.6-LS7.6-FD, B.Cu at (48.9, 43.4)
- added C6: 0.1uF, imported_components:C0805, B.Cu at (176.0, 47.4)
- added C60: RVT1V101M0607, imported_components:CAP-SMD_BD6.3-L6.6-W6.6-LS7.6-FD, B.Cu at (55.8, 43.4)
- added C61: 0.47uF, imported_components:C0805, B.Cu at (71.0, 50.0)
- added C62: 1uF, imported_components:C0805, B.Cu at (74.6, 49.8)
- added C63: 1uF, imported_components:C0805, B.Cu at (73.8, 46.8)
- added C7: RVT1H470M0607, imported_components:CAP-SMD_BD6.3-L6.6-W6.6-LS7.6-FD, B.Cu at (41.6, 36.2)
- added C8: 0.1uF, imported_components:C0805, B.Cu at (243.0, 28.2)
- added C9: 10uF, imported_components:C0805, B.Cu at (60.5, 58.9)
- added CN1: PJ-320D, imported_components:AUDIO-SMD_PJ-320D, B.Cu at (61.4, 34.8)
- added CO1: Conn_02x03_Odd_Even, imported_components:HDR-SMD_6P-P2.54-V, F.Cu at (258.8, 41.4)
- added CO2: Conn_02x03_Odd_Even, imported_components:HDR-SMD_6P-P2.54-V, F.Cu at (258.8, 50.3)
- added CO3: Conn_02x03_Odd_Even, imported_components:HDR-SMD_6P-P2.54-V, F.Cu at (269.0, 41.4)
- added CO4: Conn_02x03_Odd_Even, imported_components:HDR-SMD_6P-P2.54-V, F.Cu at (269.0, 50.3)
- added D1: SS54_C22452, imported_components:SMA_L4.4-W2.8-LS5.4-R-RD, B.Cu at (89.0, 45.8)
- added D2: LED, imported_components:LED0805-RD, B.Cu at (70.7, 27.7)
- added D3: SS54_C22452, imported_components:SMA_L4.4-W2.8-LS5.4-R-RD, B.Cu at (38.4, 49.2)
- added D4: SS54_C22452, imported_components:SMA_L4.4-W2.8-LS5.4-R-RD, B.Cu at (40.2, 43.6)
- added D5: SS54_C22452, imported_components:SMA_L4.4-W2.8-LS5.4-R-RD, B.Cu at (89.7, 58.0)
- added H1: MountingHole, MountingHole:MountingHole_3.2mm_M3_Pad_Via, F.Cu at (18.8, 96.6)
- added H2: MountingHole, MountingHole:MountingHole_3.2mm_M3_Pad_Via, F.Cu at (278.7, 96.5)
- added H3: MountingHole, MountingHole:MountingHole_3.2mm_M3_Pad_Via, F.Cu at (18.8, 28.8)
- added H4: MountingHole, MountingHole:MountingHole_3.2mm_M3_Pad_Via, F.Cu at (278.6, 28.8)
- added H5: MountingHole, MountingHole:MountingHole_3.2mm_M3_Pad_Via, F.Cu at (148.8, 62.8)
- added J1: Conn_01x02, Connector_PinHeader_2.54mm:PinHeader_1x02_P2.54mm_Vertical, B.Cu at (26.0, 27.1)
- added J2: Barrel_Jack, imported_components:DC-IN-TH_DC-005-A200, B.Cu at (34.8, 36.0)
- added J3: Conn_01x08_Pin, Connector_PinHeader_2.54mm:PinHeader_1x08_P2.54mm_Vertical, F.Cu at (17.0, 35.5)
- added J4: Conn_01x08_Pin, Connector_PinHeader_2.54mm:PinHeader_1x08_P2.54mm_Vertical, F.Cu at (280.4, 35.5)
- added L1: BLM21PG221SN1D, imported_components:L0805, B.Cu at (94.8, 45.8)
- added L2: CYA1040-33UH, imported_components:IND-SMD_L11.6-W10.1, B.Cu at (44.0, 59.0)
- added L3: BLM21PG221SN1D, imported_components:L0805, B.Cu at (95.6, 58.0)
- added LED1: SK6812MINI, imported_components:SK6812-MINI-E, B.Cu at (72.3, 33.1)
- added LED10: SK6812MINI, imported_components:SK6812-MINI-E, B.Cu at (53.3, 61.7)
- added LED11: SK6812MINI, imported_components:SK6812-MINI-E, B.Cu at (91.4, 61.7)
- added LED12: SK6812MINI, imported_components:SK6812-MINI-E, B.Cu at (110.4, 61.7)
- added LED13: SK6812MINI, imported_components:SK6812-MINI-E, B.Cu at (129.5, 61.7)
- added LED14: SK6812MINI, imported_components:SK6812-MINI-E, B.Cu at (167.6, 61.7)
- added LED15: SK6812MINI, imported_components:SK6812-MINI-E, B.Cu at (186.6, 61.7)
- added LED16: SK6812MINI, imported_components:SK6812-MINI-E, B.Cu at (224.7, 61.7)
- added LED17: SK6812MINI, imported_components:SK6812-MINI-E, B.Cu at (243.8, 61.7)
- added LED18: SK6812MINI, imported_components:SK6812-MINI-E, B.Cu at (262.8, 61.7)
- added LED19: SK6812MINI, imported_components:SK6812-MINI-E, B.Cu at (24.7, 80.7)
- added LED2: SK6812MINI, imported_components:SK6812-MINI-E, B.Cu at (91.4, 33.1)
- added LED20: SK6812MINI, imported_components:SK6812-MINI-E, B.Cu at (43.8, 80.7)
- added LED21: SK6812MINI, imported_components:SK6812-MINI-E, B.Cu at (62.8, 80.7)
- added LED22: SK6812MINI, imported_components:SK6812-MINI-E, B.Cu at (81.8, 80.7)
- added LED23: SK6812MINI, imported_components:SK6812-MINI-E, B.Cu at (100.9, 80.7)
- added LED24: SK6812MINI, imported_components:SK6812-MINI-E, B.Cu at (120.0, 80.7)
- added LED25: SK6812MINI, imported_components:SK6812-MINI-E, B.Cu at (139.0, 80.7)
- added LED26: SK6812MINI, imported_components:SK6812-MINI-E, B.Cu at (158.1, 80.7)
- added LED27: SK6812MINI, imported_components:SK6812-MINI-E, B.Cu at (177.1, 80.7)
- added LED28: SK6812MINI, imported_components:SK6812-MINI-E, B.Cu at (196.2, 80.7)
- added LED29: SK6812MINI, imported_components:SK6812-MINI-E, B.Cu at (215.2, 80.7)
- added LED3: SK6812MINI, imported_components:SK6812-MINI-E, B.Cu at (110.4, 33.1)
- added LED30: SK6812MINI, imported_components:SK6812-MINI-E, B.Cu at (234.2, 80.7)
- added LED31: SK6812MINI, imported_components:SK6812-MINI-E, B.Cu at (253.3, 80.7)
- added LED32: SK6812MINI, imported_components:SK6812-MINI-E, B.Cu at (272.4, 80.7)
- added LED33: SK6812MINI, imported_components:SK6812-MINI-E, B.Cu at (236.8, 37.8)
- added LED34: SK6812MINI, imported_components:SK6812-MINI-E, B.Cu at (243.9, 37.8)
- added LED35: SK6812MINI, imported_components:SK6812-MINI-E, B.Cu at (250.9, 37.8)
- added LED36: SK6812MINI, imported_components:SK6812-MINI-E, B.Cu at (236.8, 42.2)
- added LED37: SK6812MINI, imported_components:SK6812-MINI-E, B.Cu at (243.8, 42.2)
- added LED38: SK6812MINI, imported_components:SK6812-MINI-E, B.Cu at (250.9, 42.2)
- added LED39: SK6812MINI, imported_components:SK6812-MINI-E, B.Cu at (236.7, 46.6)
- added LED4: SK6812MINI, imported_components:SK6812-MINI-E, B.Cu at (129.5, 33.1)
- added LED40: SK6812MINI, imported_components:SK6812-MINI-E, B.Cu at (243.7, 46.6)
- added LED41: SK6812MINI, imported_components:SK6812-MINI-E, B.Cu at (250.7, 46.5)
- added LED42: SK6812MINI, imported_components:SK6812-MINI-E, B.Cu at (236.6, 50.8)
- added LED43: SK6812MINI, imported_components:SK6812-MINI-E, B.Cu at (243.6, 50.8)
- added LED44: SK6812MINI, imported_components:SK6812-MINI-E, B.Cu at (250.6, 50.8)
- added LED45: SK6812MINI, imported_components:SK6812-MINI-E, B.Cu at (257.6, 29.0)
- added LED5: SK6812MINI, imported_components:SK6812-MINI-E, B.Cu at (148.5, 33.1)
- added LED6: SK6812MINI, imported_components:SK6812-MINI-E, B.Cu at (167.6, 33.1)
- added LED7: SK6812MINI, imported_components:SK6812-MINI-E, B.Cu at (186.6, 33.1)
- added LED8: SK6812MINI, imported_components:SK6812-MINI-E, B.Cu at (205.7, 33.1)
- added LED9: SK6812MINI, imported_components:SK6812-MINI-E, B.Cu at (34.2, 61.7)
- added P1: USB_C_Plug, imported_components:USB-C_SMD-TYPE-C-31-M-12, B.Cu at (51.6, 30.7)
- added R1: 100, imported_components:R0805, B.Cu at (127.8, 46.6)
- added R10: 10k, imported_components:R0805, B.Cu at (237.2, 32.2)
- added R11: 120, imported_components:R0805, B.Cu at (17.8, 57.0)
- added R12: 100k, imported_components:R0805, B.Cu at (79.4, 36.4)
- added R13: 20k, imported_components:R0805, B.Cu at (77.8, 57.4)
- added R14: 20k, imported_components:R0805, B.Cu at (79.8, 57.4)
- added R15: 22, imported_components:R0805, B.Cu at (73.8, 44.6)
- added R16: 20k, imported_components:R0805, B.Cu at (66.6, 54.0)
- added R17: 20k, imported_components:R0805, B.Cu at (66.6, 56.0)
- added R2: 100, imported_components:R0805, B.Cu at (183.2, 46.4)
- added R3: 5.1k, imported_components:R0805, B.Cu at (48.6, 36.2)
- added R4: 5.1k, imported_components:R0805, B.Cu at (46.6, 36.2)
- added R5: 200, imported_components:R0805, B.Cu at (66.6, 27.8)
- added R6: 10k, imported_components:R0805, B.Cu at (243.0, 32.2)
- added R7: 22, imported_components:R0805, B.Cu at (217.6, 75.6)
- added R8: 22, imported_components:R0805, B.Cu at (217.6, 73.6)
- added R9: 10k, imported_components:R0805, B.Cu at (239.4, 32.2)
- added S1: GH39FKSW, imported_components:SOT-23-3_L2.9-W1.3-P1.90-LS2.4-BR, F.Cu at (72.3, 38.1)
- added S10: GH39FKSW, imported_components:SOT-23-3_L2.9-W1.3-P1.90-LS2.4-BR, F.Cu at (53.3, 66.7)
- added S11: GH39FKSW, imported_components:SOT-23-3_L2.9-W1.3-P1.90-LS2.4-BR, F.Cu at (91.4, 66.7)
- added S12: GH39FKSW, imported_components:SOT-23-3_L2.9-W1.3-P1.90-LS2.4-BR, F.Cu at (110.4, 66.7)
- added S13: GH39FKSW, imported_components:SOT-23-3_L2.9-W1.3-P1.90-LS2.4-BR, F.Cu at (129.5, 66.7)
- added S14: GH39FKSW, imported_components:SOT-23-3_L2.9-W1.3-P1.90-LS2.4-BR, F.Cu at (167.6, 66.7)
- added S15: GH39FKSW, imported_components:SOT-23-3_L2.9-W1.3-P1.90-LS2.4-BR, F.Cu at (186.6, 66.7)
- added S16: GH39FKSW, imported_components:SOT-23-3_L2.9-W1.3-P1.90-LS2.4-BR, F.Cu at (224.7, 66.7)
- added S17: GH39FKSW, imported_components:SOT-23-3_L2.9-W1.3-P1.90-LS2.4-BR, F.Cu at (243.8, 66.7)
- added S18: GH39FKSW, imported_components:SOT-23-3_L2.9-W1.3-P1.90-LS2.4-BR, F.Cu at (262.8, 66.7)
- added S19: GH39FKSW, imported_components:SOT-23-3_L2.9-W1.3-P1.90-LS2.4-BR, F.Cu at (24.7, 85.7)
- added S2: GH39FKSW, imported_components:SOT-23-3_L2.9-W1.3-P1.90-LS2.4-BR, F.Cu at (91.4, 38.1)
- added S20: GH39FKSW, imported_components:SOT-23-3_L2.9-W1.3-P1.90-LS2.4-BR, F.Cu at (43.8, 85.7)
- added S21: GH39FKSW, imported_components:SOT-23-3_L2.9-W1.3-P1.90-LS2.4-BR, F.Cu at (62.8, 85.7)
- added S22: GH39FKSW, imported_components:SOT-23-3_L2.9-W1.3-P1.90-LS2.4-BR, F.Cu at (81.8, 85.7)
- added S23: GH39FKSW, imported_components:SOT-23-3_L2.9-W1.3-P1.90-LS2.4-BR, F.Cu at (100.9, 85.7)
- added S24: GH39FKSW, imported_components:SOT-23-3_L2.9-W1.3-P1.90-LS2.4-BR, F.Cu at (120.0, 85.7)
- added S25: GH39FKSW, imported_components:SOT-23-3_L2.9-W1.3-P1.90-LS2.4-BR, F.Cu at (139.0, 85.7)
- added S26: GH39FKSW, imported_components:SOT-23-3_L2.9-W1.3-P1.90-LS2.4-BR, F.Cu at (158.1, 85.7)
- added S27: GH39FKSW, imported_components:SOT-23-3_L2.9-W1.3-P1.90-LS2.4-BR, F.Cu at (177.1, 85.7)
- added S28: GH39FKSW, imported_components:SOT-23-3_L2.9-W1.3-P1.90-LS2.4-BR, F.Cu at (196.2, 85.7)
- added S29: GH39FKSW, imported_components:SOT-23-3_L2.9-W1.3-P1.90-LS2.4-BR, F.Cu at (215.2, 85.7)
- added S3: GH39FKSW, imported_components:SOT-23-3_L2.9-W1.3-P1.90-LS2.4-BR, F.Cu at (110.4, 38.1)
- added S30: GH39FKSW, imported_components:SOT-23-3_L2.9-W1.3-P1.90-LS2.4-BR, F.Cu at (234.2, 85.7)
- added S31: GH39FKSW, imported_components:SOT-23-3_L2.9-W1.3-P1.90-LS2.4-BR, F.Cu at (253.3, 85.7)
- added S32: GH39FKSW, imported_components:SOT-23-3_L2.9-W1.3-P1.90-LS2.4-BR, F.Cu at (272.4, 85.7)
- added S4: GH39FKSW, imported_components:SOT-23-3_L2.9-W1.3-P1.90-LS2.4-BR, F.Cu at (129.5, 38.1)
- added S5: GH39FKSW, imported_components:SOT-23-3_L2.9-W1.3-P1.90-LS2.4-BR, F.Cu at (148.5, 38.1)
- added S6: GH39FKSW, imported_components:SOT-23-3_L2.9-W1.3-P1.90-LS2.4-BR, F.Cu at (167.6, 38.1)
- added S7: GH39FKSW, imported_components:SOT-23-3_L2.9-W1.3-P1.90-LS2.4-BR, F.Cu at (186.6, 38.1)
- added S8: GH39FKSW, imported_components:SOT-23-3_L2.9-W1.3-P1.90-LS2.4-BR, F.Cu at (205.7, 38.1)
- added S9: GH39FKSW, imported_components:SOT-23-3_L2.9-W1.3-P1.90-LS2.4-BR, F.Cu at (34.2, 66.7)
- added SW1: SW_SPDT, imported_components:SW-SMD_MST-12D18G4-SPDT-SLIDE-SWITCH, B.Cu at (41.6, 30.4)
- added SW2: SW_Push, imported_components:SW-SMD_L3.9-W3.0-P4.45, B.Cu at (252.8, 28.8)
- added SW3: SW_Push, imported_components:SW-SMD_L3.9-W3.0-P4.45, B.Cu at (247.8, 28.8)
- added SW4: RotaryEncoder_Switch, Rotary_Encoder:RotaryEncoder_Alps_EC11E-Switch_Vertical_H20mm, F.Cu at (217.6, 35.4)
- added U1: AMS1117-3.3, Package_TO_SOT_SMD:SOT-223-3_TabPin2, B.Cu at (100.8, 48.2)
- added U10: LM4810, Package_SO:TSSOP-8_3x3mm_P0.65mm, B.Cu at (66.8, 49.8)
- added U11: ES9023P, imported_components:SOP-16_L9.9-W3.9-P1.27-LS6.1-BL, B.Cu at (79.4, 46.2)
- added U2: 74HC4067PW,118, imported_components:TSSOP-24_L7.8-W4.4-P0.65-LS6.4-BL, B.Cu at (124.8, 52.6)
- added U3: 74HC4067PW,118, imported_components:TSSOP-24_L7.8-W4.4-P0.65-LS6.4-BL, B.Cu at (180.2, 52.5)
- added U4: AMS1117-3.3, Package_TO_SOT_SMD:SOT-223-3_TabPin2, B.Cu at (55.0, 56.0)
- added U5: ESP32-S3-WROOM-1-N4, imported_components:WIFIM-SMD_ESP32-S3-WROOM-1-N8, B.Cu at (205.8, 67.4)
- added U6: LM2596SX-5.0/NOPB, imported_components:TO-263-5_L10.2-W8.9-P1.70-TL, B.Cu at (29.6, 45.4)
- added U7: SP3485EN-L/TR, imported_components:SOIC-8_L5.0-W4.0-P1.27-LS6.0-BL, B.Cu at (72.4, 84.6)
- added U8: AMS1117-3.3, Package_TO_SOT_SMD:SOT-223-3_TabPin2, B.Cu at (73.0, 65.6)
- added U9: SX1M12.288M10F30TNN, imported_components:OSC-SMD_4P-L2.0-W1.6-BL, B.Cu at (67.5, 42.8)
Routing:
- net +3.3VA: vias 0 -> 5
- added copper zone on In2.Cu, net +3.3VA
- added copper zone on In2.Cu, net +3.3VB
- added copper zone on In1.Cu, net +5V
- added copper zone on B.Cu, net AGND
- added copper zone on F.Cu, net AGND
Other:
- board outline added: 267 x 75 mm
- copper layers 2 -> 4
- board text added: "BOOT"
- board text added: "RST"
