File: PCB/Audio Output.kicad_sch (KiCad schematic)
At the start: 74 parts, among them CN1 PJ-320D, U10 LM4810, U11 ES9023P, U8 AMS1117-3.3, U9 SX1M12.288M10F30TNN

Commit message: PCB routing done
Parts:
- renumbered LED30 to LED16, LED29 to LED17, LED28 to LED18, LED27 to LED19, LED26 to LED20, LED25 to LED21, LED24 to LED22, LED22 to LED24, LED21 to LED25, LED20 to LED26, LED19 to LED27, LED18 to LED28, LED17 to LED29, LED16 to LED30
Changed lines of the file:
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@@
 		(on_board yes)
 		(dnp no)
-		(property "Reference" "LED28"
+		(property "Reference" "LED18"
 			(at 240.792 132.334 0)
 			(effects
@@
 			(project "Fracture"
 				(path "/75221650-6511-45d6-90de-2d3fdbaa0af3/0f8c0c29-04b9-439a-a446-990ae8598d99"
-					(reference "LED28")
+					(reference "LED18")
 					(unit 1)
 				)
@@
 		(on_board yes)
 		(dnp no)
-		(property "Reference" "LED22"
+		(property "Reference" "LED24"
 			(at 141.732 132.334 0)
 			(effects
@@
 			(project "Fracture"
 				(path "/75221650-6511-45d6-90de-2d3fdbaa0af3/0f8c0c29-04b9-439a-a446-990ae8598d99"
-					(reference "LED22")
+					(reference "LED24")
 					(unit 1)
 				)
@@
 		(on_board yes)
 		(dnp no)
-		(property "Reference" "LED29"
+		(property "Reference" "LED17"
 			(at 257.302 132.334 0)
 			(effects
@@
 			(project "Fracture"
 				(path "/75221650-6511-45d6-90de-2d3fdbaa0af3/0f8c0c29-04b9-439a-a446-990ae8598d99"
-					(reference "LED29")
+					(reference "LED17")
 					(unit 1)
 				)
@@
 		(on_board yes)
 		(dnp no)
-		(property "Reference" "LED24"
+		(property "Reference" "LED22"
 			(at 174.752 132.334 0)
 			(effects
@@
 			(project "Fracture"
 				(path "/75221650-6511-45d6-90de-2d3fdbaa0af3/0f8c0c29-04b9-439a-a446-990ae8598d99"
-					(reference "LED24")
+					(reference "LED22")
 					(unit 1)
 				)
@@
 		(on_board yes)
 		(dnp no)
-		(property "Reference" "LED16"
+		(property "Reference" "LED30"
 			(at 42.672 132.334 0)
 			(effects
@@
 			(project "Fracture"
 				(path "/75221650-6511-45d6-90de-2d3fdbaa0af3/0f8c0c29-04b9-439a-a446-990ae8598d99"
-					(reference "LED16")
+					(reference "LED30")
 					(unit 1)
 				)
@@
 		(on_board yes)
 		(dnp no)
-		(property "Reference" "LED25"
+		(property "Reference" "LED21"
 			(at 191.262 132.334 0)
 			(effects
@@
 			(project "Fracture"
 				(path "/75221650-6511-45d6-90de-2d3fdbaa0af3/0f8c0c29-04b9-439a-a446-990ae8598d99"
-					(reference "LED25")
+					(reference "LED21")
 					(unit 1)
 				)
@@
 		(on_board yes)
 		(dnp no)
-		(property "Reference" "LED18"
+		(property "Reference" "LED28"
 			(at 75.692 132.334 0)
 			(effects
@@
 			(project "Fracture"
 				(path "/75221650-6511-45d6-90de-2d3fdbaa0af3/0f8c0c29-04b9-439a-a446-990ae8598d99"
-					(reference "LED18")
+					(reference "LED28")
 					(unit 1)
 				)
@@
 		(on_board yes)
 		(dnp no)
-		(property "Reference" "LED17"
+		(property "Reference" "LED29"
 			(at 59.182 132.334 0)
 			(effects
@@
 			(project "Fracture"
 				(path "/75221650-6511-45d6-90de-2d3fdbaa0af3/0f8c0c29-04b9-439a-a446-990ae8598d99"
-					(reference "LED17")
+					(reference "LED29")
 					(unit 1)
 				)
@@
 		(on_board yes)
 		(dnp no)
-		(property "Reference" "LED26"
+		(property "Reference" "LED20"
 			(at 207.772 132.334 0)
 			(effects
@@
 			(project "Fracture"
 				(path "/75221650-6511-45d6-90de-2d3fdbaa0af3/0f8c0c29-04b9-439a-a446-990ae8598d99"
-					(reference "LED26")
+					(reference "LED20")
 					(unit 1)
 				)
@@
 		(on_board yes)
 		(dnp no)
-		(property "Reference" "LED21"
+		(property "Reference" "LED25"
 			(at 125.222 132.334 0)
 			(effects
@@
 			(project "Fracture"
 				(path "/75221650-6511-45d6-90de-2d3fdbaa0af3/0f8c0c29-04b9-439a-a446-990ae8598d99"
-					(reference "LED21")
+					(reference "LED25")
 					(unit 1)
 				)
@@
 		(on_board yes)
 		(dnp no)
-		(property "Reference" "LED30"
+		(property "Reference" "LED16"
 			(at 273.812 132.334 0)
 			(effects
@@
 			(project "Fracture"
 				(path "/75221650-6511-45d6-90de-2d3fdbaa0af3/0f8c0c29-04b9-439a-a446-990ae8598d99"
-					(reference "LED30")
+					(reference "LED16")
 					(unit 1)
 				)
@@
 		(on_board yes)
 		(dnp no)
-		(property "Reference" "LED20"
+		(property "Reference" "LED26"
 			(at 108.712 132.334 0)
 			(effects
@@
 			(project "Fracture"
 				(path "/75221650-6511-45d6-90de-2d3fdbaa0af3/0f8c0c29-04b9-439a-a446-990ae8598d99"
-					(reference "LED20")
+					(reference "LED26")
 					(unit 1)
 				)
@@
 		(on_board yes)
 		(dnp no)
-		(property "Reference" "LED27"
+		(property "Reference" "LED19"
 			(at 224.282 132.334 0)
 			(effects
@@
 			(project "Fracture"
 				(path "/75221650-6511-45d6-90de-2d3fdbaa0af3/0f8c0c29-04b9-439a-a446-990ae8598d99"
-					(reference "LED27")
+					(reference "LED19")
 					(unit 1)
 				)
@@
 		(on_board yes)
 		(dnp no)
-		(property "Reference" "LED19"
+		(property "Reference" "LED27"
 			(at 92.202 132.334 0)
 			(effects
@@
 			(project "Fracture"
 				(path "/75221650-6511-45d6-90de-2d3fdbaa0af3/0f8c0c29-04b9-439a-a446-990ae8598d99"
-					(reference "LED19")
+					(reference "LED27")
 					(unit 1)
 				)

Commit message: PCB Done and Panelized!
Parts:
- added J5, J6: Conn_01x08_Pin, Connector_PinSocket_2.54mm:PinSocket_1x08_P2.54mm_Vertical, symbol Connector:Conn_01x08_Pin
Connections:
- new net: J5.1 (Pin_1), J6.1 (Pin_1)
- new net: J5.2 (Pin_2), J6.2 (Pin_2)
- new net: J5.3 (Pin_3), J6.3 (Pin_3)
- new net: J5.4 (Pin_4), J6.4 (Pin_4)
- new net: J5.5 (Pin_5), J6.5 (Pin_5)
- new net: J5.6 (Pin_6), J6.6 (Pin_6)
- new net: J5.7 (Pin_7), J6.7 (Pin_7)
- new net: J5.8 (Pin_8), J6.8 (Pin_8)
Other:
- note added: "RS-485 CONN."
